Commit message: launching two obstacles parametrically

File: ros/src/system/gazebo/mavs/mavs_description/urdf/obstacles.urdf.xacro (robot description, xacro)
@@ -1,4 +1,6 @@
 <?xml version="1.0"?>
 <robot name="obstacle" xmlns:xacro="http://www.ros.org/wiki/xacro" >
+  <xacro:arg name="idx" default="-1"/>
+  <xacro:property name="idx" value="$(arg idx)" />
   <!-- obstacles-->
   <xacro:include filename="$(find mavs_description)/urdf/obstacle.urdf.xacro"/>
@@ -9,5 +11,4 @@
   <xacro:property name="x0" value="${mavs['mavs']['obs']['x0']}" />
   <xacro:property name="y0" value="${mavs['mavs']['obs']['y0']}" />
-  <obstacle idx="0"/>
+  <obstacle idx="${idx}"/>
 </robot>
-<!--TODO add speed-->
