Commit message: worked on programmatically adding in multiple obstacles, but it does not seems to be possible to launch multiple disconnected  links inside a single robot

File: ros/src/system/gazebo/mavs/mavs_description/urdf/obstacle.urdf.xacro (robot description, xacro)
@@ -2,5 +2,5 @@
 <robot xmlns:xacro="http://www.ros.org/wiki/xacro">
   <xacro:macro name="obstacle" params="idx">
-    <link name="obstacle" type="fixed">
+    <link name="obstacle_${idx}" type="fixed">
       <inertial>
         <origin xyz="${x0[idx]} ${y0[idx]} ${length[idx]/2}" rpy="0 0 0"/>

Commit message: moving a single obstacle

File: ros/src/system/gazebo/mavs/mavs_description/urdf/obstacle.urdf.xacro (robot description, xacro)
@@ -2,5 +2,19 @@
 <robot xmlns:xacro="http://www.ros.org/wiki/xacro">
   <xacro:macro name="obstacle" params="idx">
-    <link name="obstacle_${idx}" type="fixed">
+    <!-- root link, on the ground just below the model origin -->
+    <link name="base_footprint">
+     <visual>
+        <origin xyz="0 0 0" rpy="0 0 0" />
+        <geometry>
+          <box size="0.001 0.001 0.001" />
+        </geometry>
+      </visual>
+    </link>
+    <joint name="base_link_joint" type="fixed">
+      <origin xyz="0.0 0 1.25" rpy="0 0 0" />
+      <parent link="base_footprint"/>
+      <child link="obstacle_${idx}" />
+    </joint>
+    <link name="obstacle_${idx}">
       <inertial>
         <origin xyz="${x0[idx]} ${y0[idx]} ${length[idx]/2}" rpy="0 0 0"/>
@@ -22,7 +36,14 @@
     </link>
     <gazebo>
-      <static>true</static>
       <material>Gazebo/Black</material>
+      <plugin name="object_controller" filename="libgazebo_ros_planar_move.so">
+        <commandTopic>cmd_vel</commandTopic>
+        <odometryTopic>odom</odometryTopic>
+        <odometryFrame>odom</odometryFrame>
+        <odometryRate>20.0</odometryRate>
+        <robotBaseFrame>base_footprint</robotBaseFrame>
+      </plugin>
     </gazebo>
+<!--https://answers.ros.org/question/11506/different-cmd_vel-msgs-to-multiple-robots-on-gazebo/-->
   </xacro:macro>
 </robot>

Commit message: added in a group for each obstacle

File: ros/src/system/gazebo/mavs/mavs_description/urdf/obstacle.urdf.xacro (robot description, xacro)
@@ -12,9 +12,9 @@
     </link>
     <joint name="base_link_joint" type="fixed">
-      <origin xyz="0.0 0 1.25" rpy="0 0 0" />
+      <origin xyz="0.0 0 0.01" rpy="0 0 0" />
       <parent link="base_footprint"/>
-      <child link="obstacle_${idx}" />
+      <child link="obstacle" />
     </joint>
-    <link name="obstacle_${idx}">
+    <link name="obstacle">
       <inertial>
         <origin xyz="${x0[idx]} ${y0[idx]} ${length[idx]/2}" rpy="0 0 0"/>
@@ -38,7 +38,7 @@
       <material>Gazebo/Black</material>
       <plugin name="object_controller" filename="libgazebo_ros_planar_move.so">
-        <commandTopic>obstacle/cmd_vel_${idx}</commandTopic>
-        <odometryTopic>obstacle/odom_${idx}</odometryTopic>
-        <odometryFrame>obstacle/odom_${idx}</odometryFrame>
+        <commandTopic>cmd_vel</commandTopic>
+        <odometryTopic>odom</odometryTopic>
+        <odometryFrame>odom</odometryFrame>
         <odometryRate>20.0</odometryRate>
         <robotBaseFrame>base_footprint</robotBaseFrame>

File: ros/src/system/gazebo/mavs/mavs_description/urdf/obstacles.urdf.xacro (robot description, xacro)
@@ -1,4 +1,4 @@
 <?xml version="1.0"?>
-<robot name="obstacle_0" xmlns:xacro="http://www.ros.org/wiki/xacro" >
+<robot name="obstacle" xmlns:xacro="http://www.ros.org/wiki/xacro" >
   <!-- obstacles-->
   <xacro:include filename="$(find mavs_description)/urdf/obstacle.urdf.xacro"/>

Commit message: finished first complete working version with multiple obstacles being parametrically loaded including speed

File: ros/src/system/gazebo/mavs/mavs_description/urdf/obstacle.urdf.xacro (robot description, xacro)
@@ -12,5 +12,5 @@
     </link>
     <joint name="base_link_joint" type="fixed">
-      <origin xyz="0.0 0 0.01" rpy="0 0 0" />
+      <origin xyz="0.0 0 0" rpy="0 0 0" />
       <parent link="base_footprint"/>
       <child link="obstacle" />
@@ -19,5 +19,5 @@
       <inertial>
         <origin xyz="${x0[idx]} ${y0[idx]} ${length[idx]/2}" rpy="0 0 0"/>
-        <mass value="1.0" />
+        <mass value="100.0" />
         <inertia  ixx="0.0" ixy="0.0"  ixz="0.0"  iyy="0.0"  iyz="0.0"  izz="0.0" />
       </inertial>

File: ros/src/system/gazebo/mavs/mavs_gazebo/urdf/mavs.urdf.xacro (robot description, xacro)
@@ -17,5 +17,5 @@
   <xacro:property name="psi0" value="${mavs['mavs']['X0']['psi']}" />
   <xacro:property name="scale_factor" value="${vehicle['scale_factor']}" />
-  <xacro:property name="mesh_mode" value="1"/>
+  <xacro:property name="mesh_mode" value="${vehicle['mesh_mode']}"/>
   <!-- Vehicle geometry -->
   <xacro:property name="base_link" value="${vehicle['base_link']}" />
